File: eagle-files/esp32_s20.brd (EAGLE design)
At the start: 87.3 x 99 mm, 13 parts

Commit message: [ADD] traces
Parts:
- added X4: (no value), con-ptr500:AK500/2-H
- moved JP4 6.35 mm to (58.9, 89.4)
- moved JP5 6.35 mm to (33.5, 41.2)
- moved JP6 6.35 mm to (51.3, 41.2)
- moved JP3 6.35 mm to (36.0, 89.4)
- moved U$1 6.35 mm to (47.0, 63.5)
- turned R3 to 0 degrees
Connections:
- net +5V: now also X4.2
- net GND: now also X4.1
Routing:
- net GND: track 0.00 -> 193.7 mm
- net BTN_START: track 0.00 -> 188.9 mm
- net BTN_STOP: track 0.00 -> 139.8 mm
- net LCD_D0: track 0.00 -> 90.2 mm
- net TX: track 0.00 -> 88.1 mm
- net BTN_CLBT: track 0.00 -> 85.4 mm
- net +5V: track 0.00 -> 79.6 mm
- net N: track 0.00 -> 75.4 mm
- net RX: track 0.00 -> 75.4 mm
- net LCD_RS: track 0.00 -> 68.8 mm
- net DE: track 0.00 -> 63.2 mm
- net P: track 0.00 -> 62.5 mm
- net LCD_WR: track 0.00 -> 59.6 mm
- net LCD_D6: track 0.00 -> 58.9 mm
- net 3V3: track 0.00 -> 57.6 mm
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Other:
- board size 87.3 x 99 mm -> 87.3 x 96.5 mm

Commit message: [MOD] update traces
Routing:
- net LCD_D7: track 45.3 -> 115.6 mm, vias 0 -> 2
- net LCD_D3: track 45.9 -> 104.2 mm, vias 0 -> 2
- net LCD_WR: track 59.6 -> 110.6 mm, vias 0 -> 4
- net LCD_D6: track 58.9 -> 109.6 mm, vias 0 -> 2
- net BTN_START: track 188.9 -> 143.8 mm
- net LCD_D1: track 46.1 -> 87.8 mm, vias 0 -> 2
- net LCD_RD: track 50.2 -> 85.6 mm, vias 0 -> 2
- net LCD_RS: track 68.8 -> 100.0 mm, vias 0 -> 2
- net LCD_RST: track 20.6 -> 44.8 mm, vias 0 -> 2
- net LCD_D2: track 55.5 -> 73.4 mm, vias 0 -> 2
- net GND: track 193.7 -> 210.9 mm, vias 0 -> 6
- net RX: track 75.4 -> 62.3 mm, vias 0 -> 2
- net N: track 75.4 -> 63.7 mm, vias 0 -> 4
- net P: track 62.5 -> 72.5 mm
- net +10V_S20: track 19.0 -> 26.7 mm
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