File: eagle-files/esp32_s20.sch (EAGLE design)
At the start: 13 parts

Commit message: [ADD] traces
Parts:
- added X4: (no value), con-ptr500:AK500/2-H
Connections:
- net +5V: now also X4-2.KL
- net GND: now also X4-1.KL
Changed lines of the file:
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@@
 <part name="R2" library="BeagleBone_Black_Wireless" library_urn="urn:adsk.eagle:library:6644236" deviceset="R-US_" device="0204/7" package3d_urn="urn:adsk.eagle:package:8118465/1"/>
 <part name="R3" library="BeagleBone_Black_Wireless" library_urn="urn:adsk.eagle:library:6644236" deviceset="R-US_" device="0204/7" package3d_urn="urn:adsk.eagle:package:8118465/1"/>
+<part name="X4" library="con-ptr500" library_urn="urn:adsk.eagle:library:181" deviceset="AK500/2-H" device="" package3d_urn="urn:adsk.eagle:package:9901/1"/>
 </parts>
 <sheets>
@@
 <attribute name="VALUE" x="140.97" y="92.202" size="1.778" layer="96" rot="R180"/>
 </instance>
+<instance part="X4" gate="-1" x="132.08" y="58.42" smashed="yes" rot="R180">
+<attribute name="NAME" x="133.35" y="57.531" size="1.778" layer="95"/>
+</instance>
+<instance part="X4" gate="-2" x="132.08" y="63.5" smashed="yes" rot="R180">
+<attribute name="NAME" x="133.35" y="62.611" size="1.778" layer="95"/>
+<attribute name="VALUE" x="135.89" y="67.183" size="1.778" layer="96" rot="R180"/>
+</instance>
 </instances>
 <busses>
@@
 <label x="15.24" y="83.82" size="1.27" layer="95" rot="R180" xref="yes"/>
 </segment>
+<segment>
+<pinref part="X4" gate="-1" pin="KL"/>
+<wire x1="127" y1="58.42" x2="124.46" y2="58.42" width="0.1524" layer="91"/>
+<label x="124.46" y="58.42" size="1.27" layer="95" rot="R180" xref="yes"/>
+</segment>
 </net>
 <net name="3V3" class="0">
@@
 <label x="15.24" y="76.2" size="1.27" layer="95" rot="R180" xref="yes"/>
 </segment>
+<segment>
+<pinref part="X4" gate="-2" pin="KL"/>
+<wire x1="127" y1="63.5" x2="124.46" y2="63.5" width="0.1524" layer="91"/>
+<label x="124.46" y="63.5" size="1.27" layer="95" rot="R180" xref="yes"/>
+</segment>
 </net>
